File: kicad_hiltop_moto_board/USB_Debug.sch (KiCad schematic (older format))
At the start: 14 parts, among them U13 CP2102N-A01-GQFN24

Commit message: Unused pind removed from moto board
Parts:
- C52, C55, C56: symbol Motor_Control_Board-rescue:C-device-Sensi_Board-rescue -> moto_board-rescue:C-device-Sensi_Board-rescue-Motor_Control_Board-rescue
- R76, R77, R78, R79, R80, R81, R82, R83, R84: symbol Motor_Control_Board-rescue:R-device-Sensi_Board-rescue -> moto_board-rescue:R-device-Sensi_Board-rescue-Motor_Control_Board-rescue
- U13: symbol Motor_Control_Board-rescue:CP2102N-A01-GQFN24-silabs-Sensi_Board-rescue -> moto_board-rescue:CP2102N-A01-GQFN24-silabs-Sensi_Board-rescue-Motor_Control_Board-rescue
Changed lines of the file:
@@
 EESchema Schematic File Version 4
-LIBS:Motor_Control_Board-cache
+LIBS:moto_board-cache
 EELAYER 30 0
 EELAYER END
@@
 USB_N
 $Comp
-L Motor_Control_Board-rescue:CP2102N-A01-GQFN24-silabs-Sensi_Board-rescue U13
+L moto_board-rescue:CP2102N-A01-GQFN24-silabs-Sensi_Board-rescue-Motor_Control_Board-rescue U13
 U 1 1 5C2328D1
 P 5525 3475
@@
 	5525 2325 5525 2450
 $Comp
-L Motor_Control_Board-rescue:R-device-Sensi_Board-rescue R78
+L moto_board-rescue:R-device-Sensi_Board-rescue-Motor_Control_Board-rescue R78
 U 1 1 5C3A3F19
 P 4050 3775
@@
 	2675 2875 2975 2875
 $Comp
-L Motor_Control_Board-rescue:R-device-Sensi_Board-rescue R?
+L moto_board-rescue:R-device-Sensi_Board-rescue-Motor_Control_Board-rescue R?
 U 1 1 5C3AE29F
 P 6650 3975
@@
 $EndComp
 $Comp
-L Motor_Control_Board-rescue:R-device-Sensi_Board-rescue R?
+L moto_board-rescue:R-device-Sensi_Board-rescue-Motor_Control_Board-rescue R?
 U 1 1 5C3AF9C1
 P 6650 4075
@@
 	6125 3275 7125 3275
 $Comp
-L Motor_Control_Board-rescue:R-device-Sensi_Board-rescue R83
+L moto_board-rescue:R-device-Sensi_Board-rescue-Motor_Control_Board-rescue R83
 U 1 1 5C3B4D7B
 P 7275 3175
@@
 $EndComp
 $Comp
-L Motor_Control_Board-rescue:R-device-Sensi_Board-rescue R84
+L moto_board-rescue:R-device-Sensi_Board-rescue-Motor_Control_Board-rescue R84
 U 1 1 5C3B4EF0
 P 7275 3275
@@
 	7425 3275 7575 3275
 $Comp
-L Motor_Control_Board-rescue:R-device-Sensi_Board-rescue R76
+L moto_board-rescue:R-device-Sensi_Board-rescue-Motor_Control_Board-rescue R76
 U 1 1 5C3C0EE1
 P 3125 2875
@@
 $EndComp
 $Comp
-L Motor_Control_Board-rescue:R-device-Sensi_Board-rescue R77
+L moto_board-rescue:R-device-Sensi_Board-rescue-Motor_Control_Board-rescue R77
 U 1 1 5C3C0F83
 P 3825 2625
@@
 	3825 2400 3825 2475
 $Comp
-L Motor_Control_Board-rescue:C-device-Sensi_Board-rescue C55
+L moto_board-rescue:C-device-Sensi_Board-rescue-Motor_Control_Board-rescue C55
 U 1 1 5C3C60B5
 P 5800 2225
@@
 $EndComp
 $Comp
-L Motor_Control_Board-rescue:C-device-Sensi_Board-rescue C56
+L moto_board-rescue:C-device-Sensi_Board-rescue-Motor_Control_Board-rescue C56
 U 1 1 5C3C6FB8
 P 6225 2225
@@
 NoConn ~ 6125 3575
 $Comp
-L Motor_Control_Board-rescue:C-device-Sensi_Board-rescue C?
+L moto_board-rescue:C-device-Sensi_Board-rescue-Motor_Control_Board-rescue C?
 U 1 1 5CA83BDF
 P 3475 3275
@@
 	6125 3975 6500 3975
 $Comp
-L Motor_Control_Board-rescue:R-device-Sensi_Board-rescue R?
+L moto_board-rescue:R-device-Sensi_Board-rescue-Motor_Control_Board-rescue R?
 U 1 1 5CA8BD2A
 P 6650 3875
@@
 	6125 3875 6500 3875
 $Comp
-L Motor_Control_Board-rescue:R-device-Sensi_Board-rescue R?
+L moto_board-rescue:R-device-Sensi_Board-rescue-Motor_Control_Board-rescue R?
 U 1 1 5CA8CA4A
 P 6650 3775
