File: kicad_hiltop_moto_board/moto_board.sch (KiCad schematic (older format))
At the start: 72 parts, among them J1 Conn_01x04, J10 Conn_01x01, J11 Conn_01x01, J12 Conn_01x03, J13 Conn_01x03, J2 Conn_01x04, J3 Conn_03x32_DIN41612, J4 Conn_01x04, J5 Conn_02x05_Top_Bottom, J6 Conn_01x01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

Commit message: Moto board awaiting review
Parts:
- removed J10, J11, J6, J7: Conn_01x01, Connector_PinHeader_2.54mm:PinHeader_1x01_P2.54mm_Vertical, symbol Connector:Conn_01x01
- removed J12, J13, J8, J9: Conn_01x03, Connector_PinHeader_2.54mm:PinHeader_1x03_P2.54mm_Vertical, symbol Connector:Conn_01x03
- removed R4, R5, R6, R7: 0R, Resistor_SMD:R_0603_1608Metric, symbol device:R
- removed R48: DNF, Resistor_SMD:R_0805_2012Metric, symbol device:R
- removed R49: 0R, Resistor_SMD:R_0805_2012Metric, symbol device:R
- removed TP13, TP14, TP15, TP16, TP24: Test_Point, TestPoint:TestPoint_THTPad_D1.0mm_Drill0.5mm, symbol moto_board-rescue:Test_Point-Connector-Sensi_Board-rescue-Motor_Control_Board-r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
- added J6, J7, J8, J9: Conn_01x04, Devtank_PCB_Lib:moto_board_4_pin_header, symbol Connector:Conn_01x04
- added TP13, TP14, TP15, TP16: Test_Point, TestPoint:TestPoint_THTPad_D1.0mm_Drill0.5mm, symbol Connector:Test_Point
- added TP38: Test_Point, TestPoint:TestPoint_THTPad_D1.0mm_Drill0.5mm, symbol moto_board-rescue:Test_Point-Connector-Sensi_Board-rescue-Motor_Control_Board-r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
- J2, J4: footprint Connector_Molex:Molex_Nano-Fit_105309-xx04_1x04_P2.50mm_Vertical -> Devtank_PCB_Lib:Phoenix_Contact_SPTAF_4_way_terminal_block
- R1, R13: footprint Resistor_SMD:R_0805_2012Metric -> Resistor_SMD:R_1210_3225Metric
- R2: value 0R -> DNF
Connections:
- net GND: now also J6.3 (Pin_3), J7.3 (Pin_3), J8.3 (Pin_3), J9.3 (Pin_3)
- net M_AIN1: now also J6.2 (Pin_2)
- net M_AIN2: now also J8.2 (Pin_2)
- net M_BIN1: now also J7.2 (Pin_2)
- net M_BIN2: now also J9.2 (Pin_2)
- net V5: now also J6.1 (Pin_1), J7.1 (Pin_1), J8.1 (Pin_1), J9.1 (Pin_1), TP38.1
- net AOUT1 renamed A1
- net A1: now also TP13.1
- net AOUT2 renamed A2
- net A2: now also TP14.1
- net BOUT1 renamed B1
- net B1: now also TP15.1
- net BOUT2 renamed B2
- net B2: now also TP16.1
- new net PWM_1: J6.4 (Pin_4), J8.4 (Pin_4)
- new net PWM_2: J7.4 (Pin_4), J9.4 (Pin_4)
- no-connect marks 69 -> 65
Other:
- moved on the sheet: R1, R13, TP12

Commit message: added bom
Parts:
- C13: Devtank 108-003 -> 108-006
- J1: Devtank (none) -> 741-001
- J2, J4: Devtank (none) -> 742-001
- J5: Devtank (none) -> 710-020
- R10, R11, R12, R3, R8, R9: Devtank (none) -> 101-005
- R13: Devtank (none) -> 101-008
Changed lines of the file:
@@
 F 2 "Capacitor_SMD:CP_Elec_6.3x7.7" H 22138 5725 50  0001 C CNN
 F 3 "" H 22100 5875 50  0001 C CNN
-F 4 "108-003" H 22100 5875 50  0001 C CNN "Devtank"
+F 4 "108-006" H 22100 5875 50  0001 C CNN "Devtank"
 	1    22100 5875
 	1    0    0    -1
@@
 F 2 "Resistor_SMD:R_0603_1608Metric" V 7130 9100 50  0001 C CNN
 F 3 "" H 7200 9100 50  0001 C CNN
+F 4 "101-005" H 7200 9100 50  0001 C CNN "Devtank"
 	1    7200 9100
 	0    1    1    0
@@
 F 2 "Resistor_SMD:R_0603_1608Metric" V 7130 9850 50  0001 C CNN
 F 3 "" H 7200 9850 50  0001 C CNN
+F 4 "101-005" H 7200 9850 50  0001 C CNN "Devtank"
 	1    7200 9850
 	0    1    1    0
@@
 F 2 "Resistor_SMD:R_0603_1608Metric" V 7130 9975 50  0001 C CNN
 F 3 "" H 7200 9975 50  0001 C CNN
+F 4 "101-005" H 7200 9975 50  0001 C CNN "Devtank"
 	1    7200 9975
 	0    1    1    0
@@
 F 2 "Resistor_SMD:R_0603_1608Metric" V 7130 10100 50  0001 C CNN
 F 3 "" H 7200 10100 50  0001 C CNN
+F 4 "101-005" H 7200 10100 50  0001 C CNN "Devtank"
 	1    7200 10100
 	0    1    1    0
@@
 F 2 "Resistor_SMD:R_0603_1608Metric" V 7130 10225 50  0001 C CNN
 F 3 "" H 7200 10225 50  0001 C CNN
+F 4 "101-005" H 7200 10225 50  0001 C CNN "Devtank"
 	1    7200 10225
 	0    1    1    0
@@
 F 2 "Resistor_SMD:R_0603_1608Metric" V 7130 10475 50  0001 C CNN
 F 3 "" H 7200 10475 50  0001 C CNN
+F 4 "101-005" H 7200 10475 50  0001 C CNN "Devtank"
 	1    7200 10475
 	0    1    1    0
@@
 F 2 "Devtank_PCB_Lib:Molex_8981" H 14175 9125 50  0001 C CNN
 F 3 "~" H 14175 9125 50  0001 C CNN
+F 4 "741-001" H 14175 9125 50  0001 C CNN "Devtank"
 	1    14175 9125
 	1    0    0    -1
@@
 F 2 "Resistor_SMD:R_1210_3225Metric" V 7355 7650 50  0001 C CNN
 F 3 "" H 7425 7650 50  0001 C CNN
+F 4 "101-008" H 7425 7650 50  0001 C CNN "Devtank"
 	1    7425 7650
 	1    0    0    -1
@@
 F 2 "Connector_PinHeader_2.54mm:PinHeader_2x05_P2.54mm_Vertical" H 3075 9500 50  0001 C CNN
 F 3 "~" H 3075 9500 50  0001 C CNN
+F 4 "710-020" H 3075 9500 50  0001 C CNN "Devtank"
 	1    3075 9500
 	1    0    0    -1
@@
 F 2 "Devtank_PCB_Lib:Phoenix_Contact_SPTAF_4_way_terminal_block" H 12350 9100 50  0001 C CNN
 F 3 "~" H 12350 9100 50  0001 C CNN
+F 4 "742-001" H 12350 9100 50  0001 C CNN "Devtank"
 	1    12350 9100
 	1    0    0    -1
@@
 F 2 "Devtank_PCB_Lib:Phoenix_Contact_SPTAF_4_way_terminal_block" H 12250 10125 50  0001 C CNN
 F 3 "~" H 12250 10125 50  0001 C CNN
+F 4 "742-001" H 12250 10125 50  0001 C CNN "Devtank"
 	1    12250 10125
 	1    0    0    -1
